File: LED_Wled.kicad_pcb (KiCad board)
At the start: 2 copper layers, 20 x 100 mm, 52 parts, among them J1 SWD_PORT_SKEDD, J2 Barrel_Jack, J3 LED_VOut, J4 Microphone connector, J5 LED_signal_chan, J6 Conn_01x01, J7 5V_TP, Q1 MMBT3904, Q2 AO4485, Q3 MMBT3904, Q4 AO4485, Q5 AO4485, U1 ESP32-WROOM-32, U2 TPS5450DDAR, U3 AMS1117-3.3, U4 SN74HC125DR

Commit message: update
Connections:
- U1 pad 14: LED_OUT_LS2 -> LED_VOUT_LSWS
- U1 pad 16: LED_OUT_LS3 -> unconnected-(U1-Pad16)
- U1 pad 26: LED_VOUT_LSWS -> LED_OUT_LS2
- U1 pad 27: unconnected-(U1-Pad27) -> LED_OUT_LS3
- U4 pad 1: +5V -> GND
- U4 pad 10: +5V -> GND
- U4 pad 4: +5V -> GND
Routing:
- net LED_OUT_LS2: track 15.5 -> 29.9 mm, vias 0 -> 2
- net LED_OUT_LS3: track 8.06 -> 21.5 mm, vias 0 -> 2
- net LED_VOUT_LSWS: track 21.1 -> 8.60 mm, vias 2 -> 0
- net +5V: track 58.5 -> 49.9 mm
- net +3V3: track 85.8 -> 88.1 mm
- net Net-(R1-Pad2): track 39.5 -> 41.7 mm
- net RXD: track 21.5 -> 23.7 mm
- net TXD: track 26.2 -> 28.1 mm
- net MIC: track 15.1 -> 16.6 mm
- net LED_OUT_LS1: track 23.4 -> 24.1 mm
- net GND: vias 12 -> 13

Commit message: rev2.1.0 WIP
Connections:
- net +3V3 renamed MIC_VDD
- J4 pad 4: MIC -> unconnected-(J4-Pin_4-Pad4)
- U1 pad 13: unconnected-(U1-Pad13) -> SCK
- U1 pad 16: unconnected-(U1-Pad16) -> WS
- U1 pad 29: MIC -> unconnected-(U1-IO5-Pad29)
- U1 pad 8: unconnected-(U1-Pad8) -> SD
Routing:
- net unconnected-(U1-IO5-Pad29): track 0.00 -> 16.6 mm, vias 0 -> 1
- net MIC: track 16.6 -> 0.00 mm, vias 1 -> 0

Commit message: PCB design WIP
Parts:
- removed BOOT1: Jumper, Connector_PinHeader_1.27mm:PinHeader_1x02_P1.27mm_Vertical
- removed C10, C12, C7: 0.1uF 50V, Capacitor_SMD:C_0603_1608Metric
- removed C11, C8, C9: 10uF 50V, Capacitor_SMD:C_1206_3216Metric
- added C18: 0.1uF/50V, Capacitor_SMD:C_0402_1005Metric_Pad0.74x0.62mm_HandSolder, F.Cu at (194.8, 65.4)
- added C19: 10uF/25V, Capacitor_SMD:C_0603_1608Metric_Pad1.08x0.95mm_HandSolder, F.Cu at (197.6, 65.3)
- added C20: 1uF/16V, Capacitor_SMD:C_0402_1005Metric_Pad0.74x0.62mm_HandSolder, F.Cu at (202.0, 84.6)
- added C21: 10uF/25V, Capacitor_SMD:C_0603_1608Metric_Pad1.08x0.95mm_HandSolder, F.Cu at (199.0, 85.9)
- added C22: 10uF/25V, Capacitor_SMD:C_0603_1608Metric_Pad1.08x0.95mm_HandSolder, F.Cu at (197.6, 97.1)
- added C23: 100nF/16V, Capacitor_SMD:C_0402_1005Metric_Pad0.74x0.62mm_HandSolder, F.Cu at (209.3, 85.9)
- added C24: 0.1uF 50V, Capacitor_SMD:C_0603_1608Metric, F.Cu at (200.1, 75.9)
- added C25: 0.1uF 50V, Capacitor_SMD:C_0603_1608Metric, F.Cu at (191.7, 80.7)
- added C26: 10uF 50V, Capacitor_SMD:C_1206_3216Metric, F.Cu at (198.4, 79.9)
- added C27: 10uF 50V, Capacitor_SMD:C_1206_3216Metric, F.Cu at (207.5, 78.7)
- added C28: 0.1uF 50V, Capacitor_SMD:C_0603_1608Metric, F.Cu at (208.3, 80.7)
- added D11: SM4007, Diode_SMD:D_SOD-123F, F.Cu at (200.6, 109.0)
- added D6: LESD5D5.0CT1G, Diode_SMD:D_SOD-523, F.Cu at (197.1, 94.7)
- added D7: LESD5D5.0CT1G, Diode_SMD:D_SOD-523, F.Cu at (199.5, 93.2)
- added D8: LESD5D5.0CT1G, Diode_SMD:D_SOD-523, F.Cu at (199.5, 91.7)
- added D9: 1N5819HW-7-F, Diode_SMD:D_SOD-123, F.Cu at (199.6, 96.4)
- added F1: 7.5A, Fuse:Fuse_Blade_Mini_directSolder, F.Cu at (197.1, 142.0)
- added J11: Input1, Connector_JST:JST_XH_B2B-XH-AM_1x02_P2.50mm_Vertical, F.Cu at (228.3, 18.5)
- added J12: Input1, Connector_JST:JST_XH_B2B-XH-AM_1x02_P2.50mm_Vertical, F.Cu at (218.5, 18.5)
- added J13: Input1, Connector_JST:JST_XH_B2B-XH-AM_1x02_P2.50mm_Vertical, F.Cu at (208.5, 18.5)
- added J14: Input1, Connector_JST:JST_XH_B2B-XH-AM_1x02_P2.50mm_Vertical, F.Cu at (188.7, 18.5)
- added J15: Input1, Connector_JST:JST_XH_B2B-XH-AM_1x02_P2.50mm_Vertical, F.Cu at (198.7, 18.5)
- added J8: TYPE-C-31-M-12, Connector_USB:USB_C_Receptacle_G-Switch_GT-USB-7010ASV, F.Cu at (205.8, 92.5)
- added J9: Conn_01x01, TestPoint:TestPoint_Pad_1.5x1.5mm, F.Cu at (191.8, 83.3)
- added JP1: SolderJumper_3_Open, Jumper:SolderJumper-3_P2.0mm_Open_TrianglePad1.0x1.5mm_NumberLabels, F.Cu at (193.5, 133.2)
- added JP2: SolderJumper_3_Open, Jumper:SolderJumper-3_P2.0mm_Open_TrianglePad1.0x1.5mm_NumberLabels, F.Cu at (193.5, 139.2)
- added Q6: L8050QLT1G, Package_TO_SOT_SMD:SOT-23, F.Cu at (198.0, 68.2)
- added Q7: L8050QLT1G, Package_TO_SOT_SMD:SOT-23, F.Cu at (202.0, 68.2)
- added Q8: 2N7002, Package_TO_SOT_SMD:SOT-23, F.Cu at (193.9, 95.7)
- added R12: 0R, Resistor_SMD:R_0805_2012Metric, F.Cu at (191.8, 65.4)
- added R13: 10K (NC), Resistor_SMD:R_0805_2012Metric, F.Cu at (192.2, 85.7)
- added R14: 1K, Resistor_SMD:R_0805_2012Metric, F.Cu at (195.6, 85.7)
- added R15: 47.5K, Resistor_SMD:R_0805_2012Metric, F.Cu at (202.6, 86.1)
- added R16: 22.1K, Resistor_SMD:R_0805_2012Metric, F.Cu at (199.7, 88.4)
- added R19: 10k, Resistor_SMD:R_0805_2012Metric, F.Cu at (193.1, 68.2)
- added R20: 10k, Resistor_SMD:R_0805_2012Metric, F.Cu at (206.9, 68.2)
- added R21: 0R, Resistor_SMD:R_0805_2012Metric, F.Cu at (195.1, 68.2)
- added R22: 0R, Resistor_SMD:R_0805_2012Metric, F.Cu at (205.0, 68.2)
- added R24: 100R, Resistor_SMD:R_0805_2012Metric, F.Cu at (248.5, 26.0)
- added R25: 10k, Resistor_SMD:R_0805_2012Metric, F.Cu at (190.9, 95.7)
- added R26: 10k, Resistor_SMD:R_0805_2012Metric, F.Cu at (190.9, 92.2)
- added R27: 10k, Resistor_SMD:R_0805_2012Metric, F.Cu at (196.8, 30.9)
- added R28: 1k/250mW, Resistor_SMD:R_1206_3216Metric_Pad1.30x1.75mm_HandSolder, F.Cu at (226.5, 25.1)
- added R29: 10k, Resistor_SMD:R_0805_2012Metric, F.Cu at (226.5, 30.8)
- added R30: 1k/250mW, Resistor_SMD:R_1206_3216Metric_Pad1.30x1.75mm_HandSolder, F.Cu at (216.6, 25.1)
- added R31: 10k, Resistor_SMD:R_0805_2012Metric, F.Cu at (216.6, 30.8)
- added R32: 1k/250mW, Resistor_SMD:R_1206_3216Metric_Pad1.30x1.75mm_HandSolder, F.Cu at (206.7, 25.1)
- added R33: 10k, Resistor_SMD:R_0805_2012Metric, F.Cu at (206.7, 31.0)
- added R34: 1k/250mW, Resistor_SMD:R_1206_3216Metric_Pad1.30x1.75mm_HandSolder, F.Cu at (186.9, 25.3)
- added R35: 10k, Resistor_SMD:R_0805_2012Metric, F.Cu at (186.9, 30.9)
- added SW1: TS-1187A-B-A-B, Button_Switch_SMD:SW_Push_1P1T_XKB_TS-1187A, B.Cu at (203.6, 58.7)
- added SW2: TS-1187A-B-A-B, Button_Switch_SMD:SW_Push_1P1T_XKB_TS-1187A, B.Cu at (196.1, 58.7)
- added U10: EL817, Package_DIP:DIP-4_W7.62mm, F.Cu at (212.3, 23.9)
- added U11: EL817, Package_DIP:DIP-4_W7.62mm, F.Cu at (192.5, 23.9)
- added U12: AMS1117-3.3, Package_TO_SOT_SMD:SOT-223-3_TabPin2, F.Cu at (205.4, 73.9)
- added U5: ESP32-S3-WROOM-1-N16R2, LED_Wled:XCVR_ESP32-S3-WROOM-1-N16R2, F.Cu at (199.9, 50.4)
- added U6: CP2102N-Axx-xQFN28, Package_DFN_QFN:QFN-28-1EP_5x5mm_P0.5mm_EP3.35x3.35mm, F.Cu at (195.0, 90.8)
- added U7: EL817, Package_DIP:DIP-4_W7.62mm, F.Cu at (202.4, 23.9)
- added U8: EL817, Package_DIP:DIP-4_W7.62mm, F.Cu at (232.1, 23.9)
- added U9: EL817, Package_DIP:DIP-4_W7.62mm, F.Cu at (222.2, 23.9)
- C14: value 10uF 16V -> 0.1uF 50V; footprint Capacitor_Tantalum_SMD:CP_EIA-3216-10_Kemet-I -> Capacitor_SMD:C_0603_1608Metric
- C15: value 100nF 16V -> 10uF 50V; footprint Capacitor_SMD:C_0402_1005Metric_Pad0.74x0.62mm_HandSolder -> Capacitor_SMD:C_1206_3216Metric
- C17: value 100uF 6.3V -> 100nF/16V; footprint Capacitor_SMD:C_1206_3216Metric_Pad1.33x1.80mm_HandSolder -> Capacitor_SMD:C_0402_1005Metric_Pad0.74x0.62mm_HandSolder
- C6: value 100uF 6.3V -> 10uF 50V; footprint Capacitor_Tantalum_SMD:CP_EIA-3528-12_Kemet-T_Pad1.50x2.35mm_HandSolder -> Capacitor_SMD:C_1206_3216Metric
- J1: value SWD_PORT_SKEDD -> LED_Channel_2; footprint LED_Wled:WR_WST_REDFIT_IDC_4Pin -> Connector_JST:JST_VH_B3P-VH_1x03_P3.96mm_Vertical; moved to F.Cu
- J3: value LED_VOut -> Conn_01x01; footprint Connector_PinHeader_2.54mm:PinHeader_1x02_P2.54mm_Horizontal -> TestPoint:TestPoint_Pad_1.5x1.5mm
- J4: value Microphone connector -> LED_Channel_1; footprint Connector_PinSocket_2.00mm:PinSocket_1x05_P2.00mm_Vertical -> Connector_JST:JST_VH_B3P-VH_1x03_P3.96mm_Vertical
- J5: value LED_signal_chan -> Conn_01x01; footprint Connector_PinHeader_2.54mm:PinHeader_1x03_P2.54mm_Horizontal -> TestPoint:TestPoint_Pad_1.5x1.5mm; moved to F.Cu
- J6: moved to B.Cu
- R2: value 47ohm -> 220
- R3: value 10k -> 100R
- R8: value 0ohm -> 1k/250mW; footprint Resistor_SMD:R_0805_2012Metric -> Resistor_SMD:R_1206_3216Metric_Pad1.30x1.75mm_HandSolder; moved to F.Cu
- R9: value 3.3k -> 2.74k
- U1: value ESP32-WROOM-32 -> SN74LVC2T45DCUR; footprint RF_Module:ESP32-WROOM-32 -> Package_SO:VSSOP-8_2.4x2.1mm_P0.5mm
- U4: value SN74HC125DR -> INMP441; footprint Package_SO:SOIC-14_3.9x8.7mm_P1.27mm -> LED_Wled:INMP441; moved to B.Cu
- moved R2 71.7 mm to (129.6, 72.4), turned to 0 degrees
- moved J4 71.6 mm to (240.8, 22.5), turned to -90 degrees
- moved R3 70.1 mm to (212.1, 147.8), turned to -90 degrees
- moved D1 66.4 mm to (139.7, 69.5), turned to 0 degrees
- moved R5 66.1 mm to (131.4, 74.6), turned to 180 degrees
- moved R11 64.3 mm to (133.9, 70.0)
- moved J3 64.1 mm to (191.8, 83.3)
- moved Q1 61.8 mm to (137.0, 73.6)
- moved J1 61.3 mm to (205.7, 144.5), turned to -90 degrees
- moved G*** 53.2 mm to (253.2, 59.2)
- moved R8 50.3 mm to (196.8, 25.1), turned to 90 degrees
- moved J5 24.3 mm to (207.7, 109.0), turned to 0 degrees
- moved U3 21.1 mm to (194.6, 73.9), turned to 0 degrees
- moved U1 20.3 mm to (207.5, 84.8), turned to 90 degrees
- moved J7 20.0 mm to (191.4, 109.1), turned to 0 degrees
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Connections:
- C13 pad 1: +5V -> /PSU_5V
- C14 pad 1: +5V -> GND
- C14 pad 2: GND -> +5V
- C15 pad 1: GND -> +5V
- C15 pad 2: MIC_VDD -> GND
- C16 pad 2: MIC_VDD -> CHIP_PU
- C17 pad 1: GND -> +5V
- C17 pad 2: MIC_VDD -> GND
- C2 pad 1: +5V -> /PSU_5V
- C6 pad 1: MIC_VDD -> +5V
- D3 pad 2: VIN -> Net-(D3-A)
- D5 pad 1: VIN -> /LED_POWER
- J1 pad 1: MIC_VDD -> LED_VOUT
- J1 pad 2: TXD -> LED_OUT_HS2
- J1 pad 3: RXD -> GND
- J3 pad 1: GND -> +3.3V
- J4 pad 1: GND -> LED_VOUT
- J4 pad 2: MIC_VDD -> LED_OUT_HS1
- J4 pad 3: Net-(J4-Pin_3) -> GND
- J5 pad 1: LED_OUT_HS1 -> /PSU_5V
- L1 pad 2: +5V -> /PSU_5V
- Q2 pad 1: VIN -> /LED_POWER
- Q2 pad 2: VIN -> /LED_POWER
- Q2 pad 3: VIN -> /LED_POWER
- Q4 pad 1: VIN -> /LED_POWER
- Q4 pad 2: VIN -> /LED_POWER
- Q4 pad 3: VIN -> /LED_POWER
- Q5 pad 1: VIN -> /LED_POWER
- Q5 pad 2: VIN -> /LED_POWER
- Q5 pad 3: VIN -> /LED_POWER
- R1 pad 1: MIC_VDD -> CHIP_PU
- R1 pad 2: Net-(U1-EN) -> +3V3
- R3 pad 1: Net-(U1-IO15) -> LED_OUT_HS2
- R3 pad 2: GND -> Net-(U1-A2)
- R4 pad 2: +5V -> /PSU_5V
- R6 pad 1: VIN -> /LED_POWER
- R8 pad 1: Net-(J4-Pin_3) -> Net-(R8-Pad1)
- R8 pad 2: MIC_VDD -> Input_1
- U1 pad 1: GND -> +5V
- U1 pad 2: MIC_VDD -> Net-(U1-A1)
- U1 pad 3: Net-(U1-EN) -> Net-(U1-A2)
- U1 pad 4: unconnected-(U1-SENSOR_VP-Pad4) -> GND
- U1 pad 5: unconnected-(U1-SENSOR_VN-Pad5) -> GND
- U1 pad 6: unconnected-(U1-IO34-Pad6) -> LED_OUT_LS2
- U1 pad 7: unconnected-(U1-IO35-Pad7) -> LED_OUT_LS1
- U1 pad 8: SD -> +3.3V
- U3 pad 2: MIC_VDD -> +3V3
- U4 pad 2: LED_OUT_LS1 -> +3.3V
- U4 pad 3: LED_OUT_HS1 -> SD
- U4 pad 4: GND -> SCK
- U4 pad 5: LED_OUT_LS2 -> WS
- U4 pad 6: LED_OUT_HS2 -> GND
Routing:
- net +5V: track 49.9 -> 145.5 mm, vias 4 -> 15
- net MIC_VDD: track 88.1 -> 0.00 mm, vias 2 -> 0
- net +3V3: track 0.00 -> 67.3 mm, vias 0 -> 2
- net U0TXD: track 0.00 -> 60.9 mm, vias 0 -> 3
- net U0RXD: track 0.00 -> 58.9 mm, vias 0 -> 3
- net RTS: track 0.00 -> 46.2 mm, vias 0 -> 4
- net +3.3V: track 0.00 -> 43.7 mm, vias 0 -> 1
- net DTR: track 0.00 -> 42.8 mm, vias 0 -> 2
- net Net-(U1-EN): track 41.7 -> 0.00 mm, vias 2 -> 0
- net LED_VOUT_LSWS: track 8.60 -> 47.2 mm, vias 0 -> 1
- net GPIO0: track 0.00 -> 36.4 mm, vias 0 -> 3
- net SCK: track 0.00 -> 35.9 mm, vias 0 -> 1
- net CHIP_PU: track 0.00 -> 35.7 mm, vias 0 -> 3
- net SD: track 0.00 -> 32.1 mm, vias 0 -> 2
- net LED_OUT_LS2: track 29.9 -> 0.00 mm, vias 2 -> 0
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- added copper zone on F.Cu, net /LED_POWER
- added copper zone on F.Cu, net /PSU_5V
- removed copper zone on F.Cu, net +5V
Other:
- board size 20 x 100 mm -> 20 x 105 mm
- board text added: "VBUS"
- board text removed: "+ -"
- board text removed: "+5V_OUT"
- board text removed: "GAIN TO VCC"
- board text removed: "GND"
- board text removed: "LED1 LED2 LED3"
- board text removed: "SIGNAL OUTPUT"

Commit message: removed power indicator LED, replaced some parts to basic
Parts:
- removed D1: LED_Indicator_Red, LED_SMD:LED_0805_2012Metric
- removed J14: Input1, Connector_JST:JST_XH_B2B-XH-AM_1x02_P2.50mm_Vertical
- removed Q1: MMBT3904, Package_TO_SOT_SMD:SOT-23
- removed R11, R35: 10k, Resistor_SMD:R_0805_2012Metric
- removed R2: 220, Resistor_SMD:R_0603_1608Metric
- removed R34: 1k/250mW, Resistor_SMD:R_1206_3216Metric_Pad1.30x1.75mm_HandSolder
- removed R5: 1k, Resistor_SMD:R_0603_1608Metric
- removed U11: EL817, Package_DIP:DIP-4_W7.62mm
- D4: value SMAJ26CA -> P6SSMAJ33CA
- J4: moved to B.Cu
- Q6, Q7: value L8050QLT1G -> S9013 J3
- R15: value 47.5K -> 22k
- R16: value 22.1K -> 10K
- U10, U7, U8, U9: footprint Package_DIP:DIP-4_W7.62mm -> Package_DIP:SMDIP-4_W7.62mm
- moved J4 127.6 mm to (203.7, 144.6)
- moved R24 68.4 mm to (209.0, 81.8), turned to -90 degrees
- moved R3 62.5 mm to (209.0, 85.3)
- moved J12 59.0 mm to (227.4, 76.8), turned to -90 degrees
- moved U9 55.7 mm to (218.1, 79.5), turned to 180 degrees
- moved J13 51.9 mm to (227.4, 66.9), turned to -90 degrees
- moved R30 50.0 mm to (220.8, 75.0), turned to 0 degrees
- moved J15 48.0 mm to (227.4, 57.0), turned to -90 degrees
- moved U10 46.0 mm to (218.1, 69.5), turned to 180 degrees
- moved R31 44.2 mm to (215.1, 75.0), turned to 180 degrees
- moved R32 42.3 mm to (220.8, 65.1), turned to 0 degrees
- moved U7 39.0 mm to (218.1, 59.6), turned to 180 degrees
- moved R8 38.4 mm to (220.8, 55.2), turned to 0 degrees
- moved R33 35.1 mm to (214.9, 65.1), turned to 180 degrees
- moved R27 30.4 mm to (215.0, 55.2), turned to 180 degrees
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Connections:
- U5 pad 12: P_Input_5 -> unconnected-(U5-IO8-Pad12)
- U5 pad 41_10: (no net) -> GND
- U5 pad 41_11: (no net) -> GND
- U5 pad 41_12: (no net) -> GND
- U5 pad 41_13: (no net) -> GND
- U5 pad 41_14: (no net) -> GND
- U5 pad 41_15: (no net) -> GND
- U5 pad 41_16: (no net) -> GND
- U5 pad 41_17: (no net) -> GND
- U5 pad 41_18: (no net) -> GND
- U5 pad 41_19: (no net) -> GND
- U5 pad 41_20: (no net) -> GND
- U5 pad 41_21: (no net) -> GND
Routing:
- net LED_OUT_HS1: track 0.00 -> 70.5 mm, vias 0 -> 1
- net LED_OUT_HS2: track 0.00 -> 66.7 mm, vias 0 -> 1
- net P_Input_3: track 0.00 -> 65.5 mm, vias 0 -> 2
- net P_Input_4: track 0.00 -> 57.6 mm, vias 0 -> 2
- net LED_OUT_LS1: track 0.00 -> 44.2 mm, vias 0 -> 2
- net LED_OUT_LS2: track 0.00 -> 42.5 mm, vias 0 -> 2
- net +3.3V: track 43.7 -> 85.9 mm, vias 1 -> 3
- net P_Input_1: track 0.00 -> 41.0 mm, vias 0 -> 2
- net P_Input_2: track 0.00 -> 30.6 mm, vias 0 -> 2
- net +3V3: track 67.3 -> 88.9 mm, vias 2 -> 4
- net CHIP_PU: track 35.7 -> 44.0 mm, vias 3 -> 4
- net Net-(R34-Pad1): track 8.02 -> 0.00 mm
- net Net-(R32-Pad1): track 0.00 -> 7.93 mm
- net Net-(R30-Pad1): track 0.00 -> 7.91 mm
- net Net-(R28-Pad1): track 0.00 -> 7.81 mm
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Other:
- board size 20 x 105 mm -> 40 x 111 mm
