File: LED_Wled.kicad_sch (KiCad schematic)
At the start: 53 parts, among them J1 SWD_PORT_SKEDD, J2 Barrel_Jack, J3 VIN-Out, J4 MIC_input, J5 LED_signal_chan, J6 +5V Out, Q1 AO4485, Q2 AO4485, Q3 MMBT3904, Q4 AO4485, Q5 AO4485, Q6 MMBT3904, U1 ESP32-WROOM-32, U4 SN74HC125DR

Commit message: updated parts, rdy for production?
Parts:
- C1: value (none) -> 10nF 50V; footprint (none) -> Capacitor_SMD:C_0603_1608Metric
- C10, C12, C7: value (none) -> 0.1uF 50V; footprint (none) -> Capacitor_SMD:C_0603_1608Metric
- C11, C4, C5, C8, C9: value (none) -> 10uF 50V; footprint (none) -> Capacitor_SMD:C_1206_3216Metric
- C2: value 150 uF 16V -> 220 uF 16V; JLCSMT C250092 -> C250068; JLCSMT_PKG SMD-ECAP-8.3x6.7 -> SMD,8x6.7mm; JLCSMT_Part OVZ151M1CTR-0807 -> OVK221M1CTR-0807
- D1: value (none) -> LED_Indicator_Red; footprint (none) -> LED_SMD:LED_0805_2012Metric
- D2, D6, D8: value (none) -> SS34; footprint (none) -> Diode_SMD:D_SMA
- D3: value (none) -> SM4007; footprint (none) -> Diode_SMD:D_SOD-123F
- D4: value (none) -> SMAJ26CA; footprint (none) -> Diode_SMD:D_SMA
- F1: value (none) -> Polyfuse; footprint (none) -> Fuse:Fuse_Bourns_MF-RG650
- L1: value (none) -> 22uH/5A; footprint (none) -> Inductor_SMD:L_Wuerth_WE-PD2-Typ-XL
- L2: footprint Inductor_SMD:L_Coilcraft_XxL4030 -> Inductor_SMD:L_Bourns_SRP7028A_7.3x6.6mm
- L3: value (none) -> ACM1211; footprint (none) -> userdvc:ACM1211
- R2, R4, R6, R9: value (none) -> 4.7k; footprint (none) -> Resistor_SMD:R_0603_1608Metric
- R8: value (none) -> 15k; footprint (none) -> Resistor_SMD:R_0603_1608Metric
- U1: JLCSMT C701342 -> C529577; JLCSMT_PKG SMD-38_18x25.5x3.1 -> SMD,18x25.5mm; JLCSMT_Part ESP32-WROOM-32E(8MB) -> ESP32-WROOM-32D-N8; MPN ESP32-WROOM-32E(8MB) -> ESP32-WROOM-32D-N8
- U2: value (none) -> TPS5450DDAR; footprint (none) -> Package_SO:TI_SO-PowerPAD-8
- U3: value (none) -> AMS1117-3.3; footprint (none) -> Package_TO_SOT_SMD:SOT-223-3_TabPin2

Commit message: rev2.01
Parts:
- removed C3: 22uF 16V, Capacitor_SMD:C_Elec_5x5.4, symbol Device:C_Polarized_Small
- removed D6, D8: SS34, Diode_SMD:D_SMA, symbol Device:D_Schottky
- removed D7: BZT52B15, Diode_SMD:D_SOD-123, symbol Diode:BZT52Bxx
- removed F1: Polyfuse, Fuse:Fuse_Bourns_MF-RG650, symbol Device:Polyfuse
- removed J4: MIC_input, Connector_PinHeader_2.54mm:PinHeader_1x03_P2.54mm_Horizontal, symbol Connector_Generic:Conn_01x03
- removed J6: +5V Out, Connector_PinHeader_2.54mm:PinHeader_1x02_P2.54mm_Horizontal, symbol Connector_Generic:Conn_01x02
- removed L2: 3.3 µH, 6.6 A, Inductor_SMD:L_Bourns_SRP7028A_7.3x6.6mm, symbol Device:L_Iron_Small
- removed L3: ACM1211, userdvc:ACM1211, symbol userdvc:ACM1211
- removed NT1: Net-Tie_2, NetTie:NetTie-2_SMD_Pad2.0mm, symbol Device:NetTie_2
- removed Q1: AO4485, Package_SO:SOIC-8_3.9x4.9mm_P1.27mm, symbol LED_Wled:AO4485
- removed Q6: MMBT3904, Package_TO_SOT_SMD:SOT-23, symbol Transistor_BJT:MMBT3904
- removed R4: 4.7k, Resistor_SMD:R_0603_1608Metric, symbol Device:R
- removed R8: 15k, Resistor_SMD:R_0603_1608Metric, symbol Device:R
- added C13: 220 uF 16V, Capacitor_SMD:CP_Elec_8x6.7, symbol Device:C_Polarized_Small
- added C14: 10uF 16V, Capacitor_Tantalum_SMD:CP_EIA-3216-10_Kemet-I, symbol Device:C_Polarized_Small
- added C15: 100nF 16V, Capacitor_SMD:C_0402_1005Metric_Pad0.74x0.62mm_HandSolder, symbol Device:C
- added C16: 1uF 25V, Capacitor_SMD:C_0402_1005Metric_Pad0.74x0.62mm_HandSolder, symbol Device:C
- added C17: 100uF 6.3V, Capacitor_SMD:C_1206_3216Metric_Pad1.33x1.80mm_HandSolder, symbol Device:C
- added C3: 22uF/25V, Capacitor_SMD:C_1206_3216Metric, symbol Device:C
- added J4: Microphone connector, Connector_PinSocket_2.00mm:PinSocket_1x05_P2.00mm_Vertical, symbol Connector_Generic:Conn_01x05
- added J6: Conn_01x01, TestPoint:TestPoint_Pad_1.5x1.5mm, symbol Connector_Generic:Conn_01x01
- added J7: 5V_TP, TestPoint:TestPoint_Pad_1.5x1.5mm, symbol Connector_Generic:Conn_01x01
- added Q1: MMBT3904, Package_TO_SOT_SMD:SOT-23, symbol Transistor_BJT:MMBT3904
- added R4: 10k, Resistor_SMD:R_0805_2012Metric, symbol Device:R_Small
- added R8: 0ohm, Resistor_SMD:R_0805_2012Metric, symbol Device:R_Small
- C4, C5: value 10uF 50V -> 22uF/25V; JLCSMT C13585 -> C12891; MPN CL31A106KBHNNNE -> CL31A226KAHNNNE
- C6: value 22uF 10V -> 100uF 6.3V; footprint Capacitor_Tantalum_SMD:CP_EIA-3216-10_Kemet-I -> Capacitor_Tantalum_SMD:CP_EIA-3528-12_Kemet-T_Pad1.50x2.35mm_HandSolder; JLCSMT C129272 -> C16133; JLCSMT_PKG CASE-A_3216 -> CASE-B-3528; MFR CEC(Shenzhen Zhenhua XinYun Elec) -> Kyocera AVX; MPN CA45-A-10V-22uF-K -> TAJB107K006RNJ
- J2: symbol Connector:Barrel_Jack -> Connector_Generic:Conn_01x03
- J3: value VIN-Out -> LED_VOut
- L1: value 22uH/5A -> 10uH/6.5A; JLCSMT C475917 -> C2903677; JLCSMT_PKG SMD -> SMD,10.1x11.6x4mm; MFR cjiang(Changjiang Microelectronics Tech) -> Chilisin Elec; MPN FXL1040-220-M -> BMRF00101040100MA1
- R11: footprint Resistor_SMD:R_0603_1608Metric -> Resistor_SMD:R_0805_2012Metric; JLCSMT C25804 -> C17414; JLCSMT_PKG 0603 -> 0805; JLCSMT_Part 0603WAF1002T5E -> 0805W8F1002T5E; MPN 0603WAF1002T5E -> 0805W8F1002T5E
- R2: value 4.7k -> 47ohm; JLCSMT C23162 -> C23182; JLCSMT_Part 0603WAF4701T5E -> 0603WAF470JT5E; MPN 0603WAF4701T5E -> 0603WAF470JT5E
- R9: value 4.7k -> 3.3k; symbol Device:R -> Device:R_Small; JLCSMT C23162 -> C22978; JLCSMT_Part 0603WAF4701T5E -> 0603WAF3301T5E
Connections:
- net PWR_Line is gone; now on net VIN_F+: C7.2, C8.2, D3.1 (K), D4.1 (A1)
- net VBat+ is gone; now on net VIN: J2.1 (Pin_1)
- net VBat- is gone; now on net GND: C7.1, C8.1, D4.2 (A2), J2.2 (Pin_2)
- net +3V3: now also C15.2, C16.2, C17.2, J4.2 (Pin_2), R8.2; no longer R2.2
- net +5V: now also C13.1, C14.1, J6.1 (Pin_1), Q1.3 (C), R4.2
- net GND: now also C10.1, C11.1, C12.1, C2.2, C4.1, C5.1, C9.1, J2.3 (Pin_3), J3.1 (Pin_1), Q3.2 (E), R10.2, R11.2, R9.2, U2.6 (GND), U2.9 (GNDPAD), C13.2, C14.2, C15.1, C16.1, C17.1, C3.1, J4.1 (Pin_1), J7.1 (Pin_1)
- net LED_OUT_HS1: now also J5.1 (Pin_1); no longer J5.3 (Pin_3)
- net LED_OUT_HS3: now also J5.3 (Pin_3); no longer J5.1 (Pin_1)
- net LED_VOUT: now also J3.2 (Pin_2); no longer J3.1 (Pin_1)
- net MIC: now also J4.4 (Pin_4)
- net BOOT: now reaches C1.2, U2.1 (BOOT)
- net VSENSE: now reaches R9.1, U2.4 (VSENSE)
- net VSENSE: now also R4.1
- net PH: now reaches C1.1, D2.1 (K), L1.1, U2.8 (PH)
- net VIN: now reaches D3.2 (A)
- net VIN: now also D5.1 (K), Q2.1 (S), Q2.2 (S), Q2.3 (S), Q4.1 (S), Q4.2 (S), Q4.3 (S), Q5.1 (S), Q5.2 (S), Q5.3 (S), R6.1
- net VIN_F+: now reaches C10.2, C9.2
- net VIN_F+: now also C11.2, C12.2, C4.2, C5.2, U2.7 (VIN), C3.2
- net at R11.1, R5.1: now also Q1.1 (B)
- removed net GNDPWR: C10.1, C11.1, C12.1, C2.2, C4.1, C5.1, C9.1, J3.2 (Pin_2), R9.2, U2.6 (GND), U2.9 (GNDPAD)
- removed net Vin: C11.2, C12.2, C4.2, C5.2, D5.1 (K), Q2.1 (S), Q2.2 (S), Q2.3 (S), Q4.1 (S), Q4.2 (S), Q4.3 (S), Q5.1 (S), Q5.2 (S), Q5.3 (S), R6.1, U2.7 (VIN)
- new net: Q1.2 (E), R2.2
- new net: J4.3 (Pin_3), R8.1
- no-connect marks 24 -> 25
Other:
- note added: "Active indicator"
- note added: "Input DC 5V - 15V"
- note added: "Main +5V LDO, leve-shifter Features: Reverse voltage protection Ressetable fuse"
- note added: "https://webench.ti.com/appinfo/webench/scripts/SDP.cgi?ID=89DD5F4BC01BAEF0"
- note removed: "3V3 Output indicator"
- note removed: "Main +5V for 5V/5A led strip, LDO, leve-shifter Features: Reverse voltage protection Ressetable fuse"
- note removed: "https://webench.ti.com/appinfo/webench/scripts/SDP.cgi?ID=45BCB466DE974671"
- moved on the sheet: C10, C11, C12, C6, C9, D1, J1, J3, R2

Commit message: update
Connections:
- net +5V: no longer U4.1 (1OE), U4.10 (3OE), U4.4 (2OE)
- net GND: now also U4.1 (1OE), U4.10 (3OE), U4.4 (2OE)
- net LED_OUT_LS2: now also U1.26 (IO4); no longer U1.14 (IO12)
- net LED_OUT_LS3: now also U1.27 (IO16); no longer U1.16 (IO13)
- net LED_VOUT_LSWS: now also U1.14 (IO12); no longer U1.26 (IO4)
- net MIC: now also U1.7 (IO35); no longer U1.29 (IO5)
Other:
- moved on the sheet: R3

Commit message: rev2.1.0 WIP
Parts:
- removed BOOT1: Jumper, Connector_PinHeader_1.27mm:PinHeader_1x02_P1.27mm_Vertical, symbol Connector_Generic:Conn_01x02
- removed C15: 100nF 16V, Capacitor_SMD:C_0402_1005Metric_Pad0.74x0.62mm_HandSolder, symbol Device:C
- removed C17: 100uF 6.3V, Capacitor_SMD:C_1206_3216Metric_Pad1.33x1.80mm_HandSolder, symbol Device:C
- removed J1: SWD_PORT_SKEDD, LED_Wled:WR_WST_REDFIT_IDC_4Pin, symbol LED_Wled:SWD_PORT_SKEDD
- removed J3: LED_VOut, Connector_PinHeader_2.54mm:PinHeader_1x02_P2.54mm_Horizontal, symbol Connector_Generic:Conn_01x02
- removed J4: Microphone connector, Connector_PinSocket_2.00mm:PinSocket_1x05_P2.00mm_Vertical, symbol Connector_Generic:Conn_01x05
- removed J5: LED_signal_chan, Connector_PinHeader_2.54mm:PinHeader_1x03_P2.54mm_Horizontal, symbol Connector_Generic:Conn_01x03
- removed R8: 0ohm, Resistor_SMD:R_0805_2012Metric, symbol Device:R_Small
- removed U1: ESP32-WROOM-32, RF_Module:ESP32-WROOM-32, symbol RF_Module:ESP32-WROOM-32
- removed U4: SN74HC125DR, Package_SO:SOIC-14_3.9x8.7mm_P1.27mm, symbol LED_Wled:SN74HC125DR
- added C17, C23: 100nF/16V, symbol Device:C_Small
- added C18: 0.1uF/50V, symbol Device:C_Small
- added C19, C21, C22: 10uF/25V, symbol Device:C_Small
- added C20: 1uF/16V, symbol Device:C_Small
- added D10: SK6812MINI, LED_SMD:LED_SK6812MINI_PLCC4_3.5x3.5mm_P1.75mm, symbol LED:SK6812MINI
- added D11: SM4007, Diode_SMD:D_SOD-123F, symbol Device:D_Small
- added D6, D7, D8: LESD5D5.0CT1G, Diode_SMD:D_SOD-523, symbol Diode:ESD9B3.3ST5G
- added D9: 1N5819HW-7-F, Diode_SMD:D_SOD-123, symbol Device:D_Schottky_Small
- added F1: 7.5A, symbol Device:Fuse
- added J1: LED_Channel_2, symbol Connector_Generic:Conn_01x03
- added J4: LED_Channel_1, symbol Connector_Generic:Conn_01x03
- added J8: USB_C_Receptacle_USB2.0, symbol Connector:USB_C_Receptacle_USB2.0
- added JP1: SolderJumper_3_Open, Jumper:SolderJumper-3_P2.0mm_Open_TrianglePad1.0x1.5mm_NumberLabels, symbol Jumper:SolderJumper_3_Open
- added Q6, Q7: L8050QLT1G, Package_TO_SOT_SMD:SOT-23, symbol Simulation_SPICE:NPN
- added Q8: 2N7002, Package_TO_SOT_SMD:SOT-23, symbol Transistor_FET:2N7002
- added R12, R17, R18, R21, R22, R23: 0R, Resistor_SMD:R_0805_2012Metric, symbol Device:R_Small
- added R13: 10K (NC), Resistor_SMD:R_0805_2012Metric, symbol Device:R_Small
- added R14: 1K, Resistor_SMD:R_0805_2012Metric, symbol Device:R_Small
- added R15: 47.5K, Resistor_SMD:R_0805_2012Metric, symbol Device:R_Small
- added R16: 22.1K, Resistor_SMD:R_0805_2012Metric, symbol Device:R_Small
- added R19, R20, R25, R26: 10k, Resistor_SMD:R_0805_2012Metric, symbol Device:R_Small
- added R24: 100R, Resistor_SMD:R_0805_2012Metric, symbol Device:R_Small
- added SW1, SW2: SW_Push, symbol Switch:SW_Push
- added U1: SN74LVC2T45DCUR, Package_SO:VSSOP-8_2.4x2.1mm_P0.5mm, symbol Logic_LevelTranslator:SN74LVC2T45DCUR
- added U4: INMP441, LED_Wled:INMP441, symbol LED_Wled:INMP441
- added U5: ESP32-S3-WROOM-1-N16R2, LED_Wled:XCVR_ESP32-S3-WROOM-1-N16R2, symbol LED_Wled:ESP32-S3-WROOM-1-N16R2
- added U6: CP2102N-Axx-xQFN28, Package_DFN_QFN:QFN-28-1EP_5x5mm_P0.5mm_EP3.35x3.35mm, symbol Interface_USB:CP2102N-Axx-xQFN28
- R3: value 10k -> 100R; JLCSMT C17414 -> (none); JLCSMT_PKG 0805 -> (none); JLCSMT_Part 0805W8F1002T5E -> (none); MANUFACTURER UNI-ROYAL(Uniroyal Elec) -> (none); MFR UNI-ROYAL(Uniroyal Elec) -> (none); MPN 0805W8F1002T5E -> (none)
- R9: value 3.3k -> 2.74k; JLCSMT C22978 -> (none); JLCSMT_PKG 0603 -> (none); JLCSMT_Part 0603WAF3301T5E -> (none); MANUFACTURER UNI-ROYAL(Uniroyal Elec) -> (none); MFR UNI-ROYAL(Uniroyal Elec) -> (none)
Connections:
- net +3V3: now also C21.2, C23.2, D10.4 (VDD), Q8.1 (G), R14.1, R25.2, U1.8 (VCCB), U4.2 (VDD), U6.6 (VDD), U6.7 (VREGIN); no longer C16.2, R1.1
- net +5V: now also C17.1, C22.2, D11.1 (K), D9.1 (K), JP1.1 (A), R26.2, U1.1 (VCCA); no longer C13.1, C2.1, L1.2, R4.2
- net GND: now also C16.2, R1.1, C17.2, C18.2, C19.2, C20.2, C21.1, C22.1, C23.1, D10.2 (VSS), D6.1 (A1), D7.1 (A1), D8.1 (A1), J1.1 (Pin_1), J4.1 (Pin_1), J8.A1 (GND), J8.A12 (GND), J8.B1 (GND), J8.B12 (GND), J8.S1 (SHIELD), R13.2, R15.2, R21.2, R22.2, SW1.1, SW1.2, SW2.1, SW2.2, U1.4 (GND), U1.5 (DIR), U4.1 (GND), U4.6 (L/R), U5.1 (GND), U5.27 (IO0), U5.3 (EN), U5.40 (GND), U5.41_1 (GND), U5.41_2 (GND), U5.41_3 (GND), U5.41_4 (GND), U5.41_5 (GND), U5.41_6 (GND), U5.41_7 (GND), U5.41_8 (GND), U5.41_9 (GND), U6.29 (GND), U6.3 (GND); no longer R3.2
- net LED_OUT_HS1: now also J4.2 (Pin_2), R24.1
- net LED_OUT_HS2: now also R3.1, J1.2 (Pin_2)
- net LED_OUT_LS1: now also U1.7 (B1), U5.39 (IO1)
- net LED_OUT_LS2: now also U1.6 (B2), U5.38 (IO2)
- net LED_VOUT: now also J1.3 (Pin_3), J4.3 (Pin_3)
- net LED_VOUT_HSWS: now also Q8.3 (D), R26.1
- net LED_VOUT_LSWS: now also Q8.2 (S), R25.1, U5.9 (IO16)
- net VIN: now also F1.1; no longer D3.2 (A)
- net ESP_3V3: now reaches R1.2
- net ESP_3V3: now also R12.1, U5.2 (3V3)
- new net: C13.1, C2.1, D11.2 (A), L1.2, R4.2
- new net: D3.2 (A), JP1.3 (B)
- new net: Q7.2 (B), R19.1
- new net: R14.2, U6.9 (~{RST})
- new net: R3.2, U1.3 (A2)
- new net: Q6.2 (B), R20.1
- new net: Q7.1 (C), R22.1
- new net: C20.1, R15.1, R16.1, U6.8 (VBUS)
- new net: R17.1, U6.26 (TXD)
- new net: C18.1, C19.1, R12.2
- new net: R24.2, U1.2 (A1)
- new net: F1.2, JP1.2 (C)
- new net: R13.1, U6.11 (~{SUSPEND})
- new net: R18.1, U6.25 (RXD)
- new net: Q6.1 (C), R21.1
- new net: D10.3 (DIN), R23.2
- new net DTR: Q6.3 (E), R19.2, U6.28 (~{DTR})
- new net GPIO10: U5.18 (IO10)
- new net GPIO11: U5.19 (IO11)
- new net GPIO12: U5.20 (IO12)
- new net GPIO17: U5.10 (IO17)
- new net GPIO18: U5.11 (IO18)
- new net GPIO19: U5.13 (IO19)
- new net GPIO20: U5.14 (IO20)
- new net GPIO21: U5.23 (IO21)
- new net GPIO3: U5.15 (IO3)
- new net GPIO35: U5.28 (IO35)
- new net GPIO36: U5.29 (IO36)
- new net GPIO37: U5.30 (IO37)
- new net GPIO38: R23.1, U5.31 (IO38)
- new net GPIO39: U5.32 (IO39)
- new net GPIO4: U5.4 (IO4)
- new net GPIO40: U5.33 (IO40)
- new net GPIO41: U5.34 (IO41)
- new net GPIO42: U5.35 (IO42)
- new net GPIO45: U5.26 (IO45)
- new net GPIO46: U5.16 (IO46)
- new net GPIO47: U5.24 (IO47)
- new net GPIO48: U5.25 (IO48)
- new net GPIO5: U5.5 (IO5)
- new net GPIO6: U5.6 (IO6)
- new net GPIO7: U5.7 (IO7)
- new net GPIO8: U5.12 (IO8)
- new net GPIO9: U5.17 (IO9)
- new net RTS: Q7.3 (E), R20.2, U6.24 (~{RTS})
- new net SCK: U4.4 (SCK), U5.22 (IO14)
- new net SD: U4.3 (SD), U5.21 (IO13)
- new net U0RXD: R17.2, U5.36 (RXD0)
- new net U0TXD: R18.2, U5.37 (TXD0)
- new net USB_DN: D7.2 (A2), J8.A7 (D-), J8.B7 (D-), U6.5 (D-)
- new net USB_DP: D8.2 (A2), J8.A6 (D+), J8.B6 (D+), U6.4 (D+)
- new net VBUS: D6.2 (A2), D9.2 (A), J8.A4 (VBUS), J8.A9 (VBUS), J8.B4 (VBUS), J8.B9 (VBUS), R16.2
- new net WS: U4.5 (WS), U5.8 (IO15)
- no-connect marks 25 -> 21
Other:
- note added: "J2Barell jack compatible with 5.5x2.1mm jack J3 JST-SM 2pin pigtail (optional 2 horizontal pin headers 2.54mm)"
- note added: "Level shifter To turn on relay to power LED strip"
- note added: "Microphone"
- note removed: "J1 Programming port SKEDD J2Barell jack compatible with 5.5x2.1mm jack J3 JST-SM 3pin pigtail (optional 3 horizontal pin headers 2.54mm) J4 MIC input"
- note removed: "MCU"
- moved on the sheet: C1, C10, C11, C12, C13, C14, C16, C2, C3, C4, C5, C6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

Commit message: added couple of footprints
Parts:
- C17, C18, C20, C23: footprint (none) -> Capacitor_SMD:C_0402_1005Metric_Pad0.74x0.62mm_HandSolder
- C19, C21, C22: footprint (none) -> Capacitor_SMD:C_0603_1608Metric_Pad1.08x0.95mm_HandSolder
- F1: footprint (none) -> Fuse:Fuse_Blade_Mini_directSolder
- J8: value USB_C_Receptacle_USB2.0 -> TYPE-C-31-M-12; footprint (none) -> Connector_USB:USB_C_Receptacle_G-Switch_GT-USB-7010ASV; JLCPCB_PART (none) -> C165948
- SW1, SW2: value SW_Push -> TS-1187A-B-A-B; footprint (none) -> Button_Switch_SMD:SW_Push_1P1T_XKB_TS-1187A; JLC_PART (none) -> C318884
Changed lines of the file:
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@@
       (effects (font (size 1.27 1.27)))
     )
-    (property "Footprint" "" (at 73.66 158.75 0)
+    (property "Footprint" "Capacitor_SMD:C_0402_1005Metric_Pad0.74x0.62mm_HandSolder" (at 73.66 158.75 0)
       (effects (font (size 1.27 1.27)) hide)
     )
@@
       (effects (font (size 1.27 1.27)))
     )
-    (property "Value" "SW_Push" (at 179.07 175.26 0)
-      (effects (font (size 1.27 1.27)))
-    )
-    (property "Footprint" "" (at 179.07 173.99 0)
+    (property "Value" "TS-1187A-B-A-B" (at 179.07 175.26 0)
+      (effects (font (size 1.27 1.27)))
+    )
+    (property "Footprint" "Button_Switch_SMD:SW_Push_1P1T_XKB_TS-1187A" (at 179.07 173.99 0)
       (effects (font (size 1.27 1.27)) hide)
     )
     (property "Datasheet" "~" (at 179.07 173.99 0)
+      (effects (font (size 1.27 1.27)) hide)
+    )
+    (property "JLC_PART" "C318884" (at 179.07 179.07 0)
       (effects (font (size 1.27 1.27)) hide)
     )
@@
       (effects (font (size 1.27 1.27)))
     )
-    (property "Footprint" "" (at 83.82 158.75 0)
+    (property "Footprint" "Capacitor_SMD:C_0402_1005Metric_Pad0.74x0.62mm_HandSolder" (at 83.82 158.75 0)
       (effects (font (size 1.27 1.27)) hide)
     )
@@
       (effects (font (size 1.27 1.27)))
     )
-    (property "Value" "SW_Push" (at 179.07 158.75 0)
-      (effects (font (size 1.27 1.27)))
-    )
-    (property "Footprint" "" (at 179.07 157.48 0)
+    (property "Value" "TS-1187A-B-A-B" (at 179.07 158.75 0)
+      (effects (font (size 1.27 1.27)))
+    )
+    (property "Footprint" "Button_Switch_SMD:SW_Push_1P1T_XKB_TS-1187A" (at 179.07 157.48 0)
       (effects (font (size 1.27 1.27)) hide)
     )
     (property "Datasheet" "~" (at 179.07 157.48 0)
+      (effects (font (size 1.27 1.27)) hide)
+    )
+    (property "JLC_PART" "C318884" (at 179.07 162.56 0)
       (effects (font (size 1.27 1.27)) hide)
     )
@@
       (effects (font (size 1.27 1.27)) (justify left))
     )
-    (property "Footprint" "" (at 67.31 91.44 0)
+    (property "Footprint" "Capacitor_SMD:C_0402_1005Metric_Pad0.74x0.62mm_HandSolder" (at 67.31 91.44 0)
       (effects (font (size 1.27 1.27)) hide)
     )
@@
       (effects (font (size 1.27 1.27)) (justify left))
     )
-    (property "Footprint" "" (at 299.72 73.66 0)
+    (property "Footprint" "Capacitor_SMD:C_0603_1608Metric_Pad1.08x0.95mm_HandSolder" (at 299.72 73.66 0)
       (effects (font (size 1.27 1.27)) hide)
     )
@@
       (effects (font (size 1.27 1.27)))
     )
-    (property "Value" "USB_C_Receptacle_USB2.0" (at 196.85 68.58 0)
-      (effects (font (size 1.27 1.27)))
-    )
-    (property "Footprint" "" (at 177.8 72.39 0)
+    (property "Value" "TYPE-C-31-M-12" (at 196.85 68.58 0)
+      (effects (font (size 1.27 1.27)))
+    )
+    (property "Footprint" "Connector_USB:USB_C_Receptacle_G-Switch_GT-USB-7010ASV" (at 177.8 72.39 0)
       (effects (font (size 1.27 1.27)) hide)
     )
     (property "Datasheet" "https://www.usb.org/sites/default/files/documents/usb_type-c.zip" (at 177.8 72.39 0)
+      (effects (font (size 1.27 1.27)) hide)
+    )
+    (property "JLCPCB_PART" "C165948" (at 177.8 68.58 0)
       (effects (font (size 1.27 1.27)) hide)
     )
@@
       (effects (font (size 1.27 1.27)) (justify left))
     )
-    (property "Footprint" "" (at 289.56 73.66 0)
+    (property "Footprint" "Capacitor_SMD:C_0402_1005Metric_Pad0.74x0.62mm_HandSolder" (at 289.56 73.66 0)
       (effects (font (size 1.27 1.27)) hide)
     )
@@
       (effects (font (size 1.27 1.27)))
     )
-    (property "Footprint" "" (at 63.5 260.858 90)
+    (property "Footprint" "Fuse:Fuse_Blade_Mini_directSolder" (at 63.5 260.858 90)
       (effects (font (size 1.27 1.27)) hide)
     )
@@
       (effects (font (size 1.27 1.27)) (justify left))
     )
-    (property "Footprint" "" (at 165.1 127 0)
+    (property "Footprint" "Capacitor_SMD:C_0603_1608Metric_Pad1.08x0.95mm_HandSolder" (at 165.1 127 0)
       (effects (font (size 1.27 1.27)) hide)
     )
@@
       (effects (font (size 1.27 1.27)) (justify left))
     )
-    (property "Footprint" "" (at 109.22 50.8 0)
-      (effects (font (size 1.27 1.27)) hide)
-    )
+    (property "Footprint" "Capacitor_SMD:C_0603_1608Metric_Pad1.08x0.95mm_HandSolder" (at 109.22 50.8 0)
+      (effects (font (size 1.27 1.27)) hide)
+    )
