File: LED_Wled.kicad_sch (KiCad schematic)
At the start: 83 parts, among them J1 LED_Channel_2, J2 Barrel_Jack, J4 LED_Channel_1, J6 Conn_01x01, J7 5V_TP, J8 TYPE-C-31-M-12, Q1 MMBT3904, Q2 AO4485, Q3 MMBT3904, Q4 AO4485, Q5 AO4485, Q6 L8050QLT1G, Q7 L8050QLT1G, Q8 2N7002, SW1 TS-1187A-B-A-B, SW2 TS-1187A-B-A-B, U1 SN74LVC2T45DCUR, U2 TPS5450DDAR, U3 AMS1117-3.3, U4 INMP441, U5 ESP32-S3-WROOM-1-N16R2, U6 CP2102N-Axx-xQFN28

Commit message: PCB design WIP
Parts:
- removed C10, C12, C7: 0.1uF 50V, Capacitor_SMD:C_0603_1608Metric, symbol Device:C
- removed C11, C8, C9: 10uF 50V, Capacitor_SMD:C_1206_3216Metric, symbol Device:C
- removed C14: 10uF 16V, Capacitor_Tantalum_SMD:CP_EIA-3216-10_Kemet-I, symbol Device:C_Polarized_Small
- removed C6: 100uF 6.3V, Capacitor_Tantalum_SMD:CP_EIA-3528-12_Kemet-T_Pad1.50x2.35mm_HandSolder, symbol Device:C_Polarized_Small
- removed D10: SK6812MINI, LED_SMD:LED_SK6812MINI_PLCC4_3.5x3.5mm_P1.75mm, symbol LED:SK6812MINI
- removed R17, R18, R23: 0R, Resistor_SMD:R_0805_2012Metric, symbol Device:R_Small
- added C14, C24, C25, C28: 0.1uF 50V, Capacitor_SMD:C_0603_1608Metric, symbol Device:C
- added C15, C26, C27, C6: 10uF 50V, Capacitor_SMD:C_1206_3216Metric, symbol Device:C
- added J11, J12, J13, J14, J15: Input1, Connector_JST:JST_XH_B2B-XH-AM_1x02_P2.50mm_Vertical, symbol Connector_Generic:Conn_01x02
- added J3, J5, J9: Conn_01x01, TestPoint:TestPoint_Pad_1.5x1.5mm, symbol Connector_Generic:Conn_01x01
- added JP2: SolderJumper_3_Open, Jumper:SolderJumper-3_P2.0mm_Open_TrianglePad1.0x1.5mm_NumberLabels, symbol Jumper:SolderJumper_3_Open
- added R27, R29, R31, R33, R35: 10k, Resistor_SMD:R_0805_2012Metric, symbol Device:R_Small
- added R28, R30, R32, R34, R8: 1k/250mW, Resistor_SMD:R_1206_3216Metric_Pad1.30x1.75mm_HandSolder, symbol Device:R_Small
- added U10, U11, U7, U8, U9: EL817, Package_DIP:DIP-4_W7.62mm, symbol Isolator:EL817
- added U12: AMS1117-3.3, Package_TO_SOT_SMD:SOT-223-3_TabPin2, symbol Regulator_Linear:AMS1117-3.3
- J1, J4: footprint (none) -> Connector_JST:JST_VH_B3P-VH_1x03_P3.96mm_Vertical; JLC_PART (none) -> C703273
- R2: value 47ohm -> 220; JLCSMT C23182 -> (none); JLCSMT_PKG 0603 -> (none); JLCSMT_Part 0603WAF470JT5E -> (none); MANUFACTURER UNI-ROYAL(Uniroyal Elec) -> (none); MFR UNI-ROYAL(Uniroyal Elec) -> (none); MPN 0603WAF470JT5E -> (none)
- R9: MPN 0603WAF4701T5E -> (none)
- U3: symbol Regulator_Linear:LM1117-3.3 -> Regulator_Linear:AMS1117-3.3
Connections:
- net ESP_3V3 is gone; now on net +3V3: R1.2, R12.1, U5.2 (3V3)
- net +3V3: now also C24.2, C26.1, J9.1 (Pin_1); no longer C23.2, Q8.1 (G), R25.2, U1.8 (VCCB), U4.2 (VDD)
- net +5V: now also C14.2, C15.1, C25.2, C6.1, JP2.3 (B), U12.3 (VI)
- net GND: now also J1.3 (Pin_3), J4.3 (Pin_3), C14.1, C15.2, C24.1, C25.1, C26.2, C27.2, C28.1, C6.2, R27.2, R29.2, R31.2, R33.2, R35.2, U12.1 (GND); no longer C16.2, J1.1 (Pin_1), J4.1 (Pin_1), R1.1, R21.2, R22.2, SW1.2, SW2.2, U5.27 (IO0), U5.3 (EN)
- net LED_VOUT: now also J1.1 (Pin_1), J4.1 (Pin_1); no longer J1.3 (Pin_3), J4.3 (Pin_3)
- net U0RXD: now also U6.26 (TXD)
- net U0TXD: now also U6.25 (RXD)
- net VIN: no longer D5.1 (K), Q2.1 (S), Q2.2 (S), Q2.3 (S), Q4.1 (S), Q4.2 (S), Q4.3 (S), Q5.1 (S), Q5.2 (S), Q5.3 (S), R6.1
- net VIN_F+: now also JP2.1 (A)
- net PSU_5V: now reaches C13.1, C2.1, D11.2 (A), L1.2, R4.2
- net PSU_5V: now also J5.1 (Pin_1)
- net GPIO10: no longer names the net of U5.18 (IO10)
- net GPIO11: no longer names the net of U5.19 (IO11)
- net GPIO12: no longer names the net of U5.20 (IO12)
- net GPIO17: no longer names the net of U5.10 (IO17)
- net GPIO18: no longer names the net of U5.11 (IO18)
- net GPIO19: no longer names the net of U5.13 (IO19)
- net GPIO20: no longer names the net of U5.14 (IO20)
- net GPIO21: no longer names the net of U5.23 (IO21)
- net GPIO3: no longer names the net of U5.15 (IO3)
- net GPIO35: no longer names the net of U5.28 (IO35)
- net GPIO36: no longer names the net of U5.29 (IO36)
- net GPIO37: no longer names the net of U5.30 (IO37)
- net GPIO38: no longer names the net of U5.31 (IO38)
- net GPIO39: no longer names the net of U5.32 (IO39)
- net GPIO4 renamed P_Input_1
- net P_Input_1: now also R27.1, U7.3
- net GPIO40: no longer names the net of U5.33 (IO40)
- net GPIO41: no longer names the net of U5.34 (IO41)
- net GPIO42: no longer names the net of U5.35 (IO42)
- net GPIO45: no longer names the net of U5.26 (IO45)
- net GPIO46: no longer names the net of U5.16 (IO46)
- net GPIO47: no longer names the net of U5.24 (IO47)
- net GPIO48: no longer names the net of U5.25 (IO48)
- net GPIO5 renamed P_Input_2
- net P_Input_2: now also R29.1, U8.3
- net GPIO6 renamed P_Input_3
- net P_Input_3: now also R31.1, U9.3
- net GPIO7 renamed P_Input_4
- net P_Input_4: now also R33.1, U10.3
- net GPIO8 renamed P_Input_5
- net P_Input_5: now also R35.1, U11.3
- net GPIO9: no longer names the net of U5.17 (IO9)
- new net: R30.1, U9.1
- new net: R8.1, U7.1
- new net: R28.1, U8.1
- new net: R32.1, U10.1
- new net: R34.1, U11.1
- new net +3.3V: C23.2, C27.1, C28.2, J3.1 (Pin_1), Q8.1 (G), R25.2, U1.8 (VCCB), U10.4, U11.4, U12.2 (VO), U4.2 (VDD), U7.4, U8.4, U9.4
- new net CHIP_PU: C16.2, R1.1, R22.2, SW2.2, U5.3 (EN)
- new net GPIO0: R21.2, SW1.2, U5.27 (IO0)
- new net Input_1: J15.1 (Pin_1), R8.2
- new net Input_1_GND: J15.2 (Pin_2), U7.2
- new net Input_2: J11.1 (Pin_1), R28.2
- new net Input_2_GND: J11.2 (Pin_2), U8.2
- new net Input_3: J12.1 (Pin_1), R30.2
- new net Input_3_GND: J12.2 (Pin_2), U9.2
- new net Input_4: J13.1 (Pin_1), R32.2
- new net Input_4_GND: J13.2 (Pin_2), U10.2
- new net Input_5: J14.1 (Pin_1), R34.2
- new net Input_5_GND: J14.2 (Pin_2), U11.2
- new net LED_POWER: D5.1 (K), JP2.2 (C), Q2.1 (S), Q2.2 (S), Q2.3 (S), Q4.1 (S), Q4.2 (S), Q4.3 (S), Q5.1 (S), Q5.2 (S), Q5.3 (S), R6.1
- no-connect marks 21 -> 42
Other:
- note added: "3.3V LDO for other hardware"
- note added: "JP1 for 5v or 12/24v strip"
- note added: "Main +5.7V LDO, leve-shifter Features: Reverse voltage protection Ressetable fuse"
- note removed: "Main +5V LDO, leve-shifter Features: Reverse voltage protection Ressetable fuse"
- moved on the sheet: J6, J7, U3
